File: hardware/scaner_v1/scaner_v1.kicad_sch (KiCad schematic)
At the start: 43 parts, among them J1 OBD кабель, Q1 IRFB4110, U1 LM2596S-ADJ, U2 SN65HVD230, U3 SN65HVD230, U4 XIAO_ESP32C5

Commit message: Board v1: single-sided hand routing, 4-pin CAN connector, 3D models
- Tracks on bottom copper only, no wire jumpers; routes kept in
  tools/routes.py and laid by tools/hand_route.py, DRC clean
- THT pads 2.0 mm, 0.6 mm drills, SOIC pads 0.8 mm, solid GND pour
  with 1 mm clearance, no copper under the inductor
- J2 and J3 merged into one 4-pin CAN connector
- 12x12 inductor footprint with wide pads; VRML models for the XIAO
  on sockets, inductor, fuse holder and wire leads
- Firmware: new CAN pin map, TX held high and Rs released only after
  the controller starts (no pull-ups on the board)

Co-Authored-By: Claude Opus 5.5 <noreply@anthropic.com>
Parts:
- removed D1: 1.5KE27A, Diode_THT:D_DO-201AD_P5.08mm_Vertical_AnodeUp, symbol Device:D_Zener
- removed H2: M3, MountingHole:MountingHole_3.2mm_M3, symbol Mechanical:MountingHole
- removed J1: OBD кабель, Connector_PinHeader_2.54mm:PinHeader_1x07_P2.54mm_Vertical, symbol Connector_Generic:Conn_01x07
- removed JP2: TERM_A, Jumper:SolderJumper-2_P1.3mm_Open_RoundedPad1.0x1.5mm, symbol Jumper:SolderJumper_2_Open
- removed R6: 10k, Resistor_SMD:R_0805_2012Metric, symbol Device:R
- removed U4: XIAO_ESP32C5, scaner:XIAO_ESP32C5_Socket, symbol scaner:XIAO_ESP32C5
- added C5: 10u, Capacitor_SMD:C_1206_3216Metric, symbol Device:C
- added C7: 100n, Capacitor_SMD:C_1206_3216Metric, symbol Device:C
- added J1: OBD питание, Connector_PinHeader_2.54mm:PinHeader_1x03_P2.54mm_Vertical, symbol Connector_Generic:Conn_01x03
- added J2: OBD 14 6 8 3, Connector_PinHeader_2.54mm:PinHeader_1x04_P2.54mm_Vertical, symbol Connector_Generic:Conn_01x04
- C2, C4, C6, C8: footprint Capacitor_SMD:C_0805_2012Metric -> Capacitor_SMD:C_1206_3216Metric
- D3, D4, D5: footprint Diode_THT:D_DO-35_SOD27_P2.54mm_Vertical_AnodeUp -> Diode_THT:D_DO-35_SOD27_P7.62mm_Horizontal
- D8: footprint Diode_THT:D_DO-201AD_P5.08mm_Vertical_AnodeUp -> Diode_THT:D_DO-201AD_P12.70mm_Horizontal
- H2: renamed from C7; value 100n -> M3; footprint Capacitor_SMD:C_0805_2012Metric -> MountingHole:MountingHole_3.2mm_M3; symbol Device:C -> Mechanical:MountingHole
- JP2: renamed from U2; value SN65HVD230 -> TERM_A; footprint Package_SO:SOIC-8_3.9x4.9mm_P1.27mm -> Jumper:SolderJumper-2_P1.3mm_Open_RoundedPad1.0x1.5mm; symbol Interface_CAN_LIN:SN65HVD230 -> Jumper:SolderJumper_2_Open
- L1: footprint Inductor_SMD:L_12x12mm_H4.5mm -> scaner:L_12x12mm_WidePads
- R10, R11, R12, R2, R3, R4, R7, R8: footprint Resistor_SMD:R_0805_2012Metric -> Resistor_SMD:R_1206_3216Metric
- U2: renamed from R5; value 10k -> SN65HVD230; footprint Resistor_SMD:R_0805_2012Metric -> Package_SO:SOIC-8_3.9x4.9mm_P1.27mm; symbol Device:R -> Interface_CAN_LIN:SN65HVD230
- U4: renamed from C5; value 10u -> XIAO_ESP32C5; footprint Capacitor_SMD:C_0805_2012Metric -> scaner:XIAO_ESP32C5_Socket; symbol Device:C -> scaner:XIAO_ESP32C5
Connections:
- net +3V3: now also U2.3 (VCC), U4.12 (3V3), C7.1; no longer H2.1, JP2.3 (VCC), U2.1
- net CANA_H: now also U2.7 (CANH), J2.2 (Pin_2); no longer JP2.7 (CANH)
- net CANA_L: now also JP2.2 (B), U2.6 (CANL), J2.1 (Pin_1); no longer JP2.6 (CANL)
- net CANA_RX: now also U2.4 (R), U4.8 (D7/GPIO12/RX); no longer JP2.4 (R)
- net CANA_TX: now also U2.1 (D), U4.9 (D8/GPIO8); no longer JP2.1 (D), U2.2
- net CANB_H: now also J2.4 (Pin_4)
- net CANB_L: now also J2.3 (Pin_3)
- net CANB_RX: now also U4.11 (D10/GPIO10)
- net CANB_TX: now also U4.2 (D1/GPIO0)
- net GND: now also U2.2 (GND), U4.13 (GND), C5.2, C7.2, J1.2 (Pin_2), J1.3 (Pin_3); no longer H2.2, JP2.2 (GND), U4.2
- net RS_A: now also U2.8 (Rs), U4.10 (D9/GPIO9); no longer JP2.8 (Rs)
- net RS_B: now also U4.6 (D5/GPIO24/SCL)
- net TERM_A: now also JP2.1 (A)
- net V5: now also U4.14 (5V), C5.1; no longer U4.1
- net VBAT_ADC: now also U4.1 (D0/GPIO1/A0)
- net VBAT_OBD: now also J1.1 (Pin_1)
Other:
- note added: "U2/U3 — SN65HVD230, выпаянные с модулей Waveshare. Rs: 1 (подтяжка) = только слушать, передатчик выключен; прошивка опускает в 0"
- note added: "Не занимать: D2, D3 (strapping), D6 (лог загрузки). Свободна D4"
- note added: "Повторитель Q1 ограничивает вход LM2596 ~26,5 В (IRFB4110 держит до 100 В)"
- note added: "Провода от выводов разъёма OBD: J1 1 = OBD16 (+12 В), 2 = OBD4, 3 = OBD5; J2 (у трансиверов) 1 = OBD14, 2 = OBD6, 3 = OBD8, 4 = OBD3"
- note removed: "D1 1.5KE27A — опция, по умолчанию не ставится (DNP). Повторитель Q1 ограничивает вход LM2596 ~26,5 В"
- note removed: "J1 — короткие провода от выводов разъёма в корпусе OBD: 1 = OBD16 (+12 В), 2 = OBD4, 3 = OBD5, 4 = OBD6, 5 = OBD14, 6 = OBD3, 7 = OBD8"
- note removed: "U2/U3 — SN65HVD230, выпаянные с модулей Waveshare. Rs: 1 (подтяжка) = только слушать, прошивка опускает в 0"
- note removed: "Не занимать: D2, D3 (strapping), D6 (лог загрузки). D4/D5 — Rs трансиверов, D7 — резерв"
